Commit message: crom_description: setting kinect link and camera names

File: crom_description/urdf/head/head.urdf.xacro (robot description, xacro)
@@ -189,5 +189,6 @@
 			<parent link="${name}_camera_structure_link"/>
 			<child link="${name}_kinect_link"/>
-			<origin xyz="0.030 0.0325 0.0525" rpy="0 0 0" />
+			<!-- origin xyz="0.030 0.0325 0.0525" rpy="0 0 0" (for real robot) /-->
+			<origin xyz="0.0 0.0 0.0" rpy="0 0 0" />
 			<axis xyz="0 0 1" rpy="0 0 0" />
 		</joint>
