Commit message: crom_description: modifying colours

File: crom_description/urdf/arms/lwa4p/lwa4p.gazebo.xacro (robot description, xacro)
@@ -3,35 +3,35 @@
 	<xacro:macro name="schunk_lwa4p_gazebo" params="name">
 		<gazebo reference="${name}_0_link">
-			<material value="Schunk/LightGrey" />
+			<material>Schunk/LightGrey</material>
 			<turnGravityOff>false</turnGravityOff>
             <selfCollide>true</selfCollide>
 		</gazebo>
 		<gazebo reference="${name}_1_link">
-			<material value="Schunk/Blue" />
+			<material>Schunk/Blue</material>
 			<turnGravityOff>false</turnGravityOff>
             <selfCollide>true</selfCollide>
 		</gazebo>
 		<gazebo reference="${name}_2_link">
-			<material value="Schunk/LightGrey" />
+			<material>Schunk/LightGrey</material>
 			<turnGravityOff>false</turnGravityOff>
             <selfCollide>true</selfCollide>
 		</gazebo>
 		<gazebo reference="${name}_3_link">
-			<material value="Schunk/Blue" />
+			<material>Schunk/Blue</material>
 			<turnGravityOff>false</turnGravityOff>
              <selfCollide>true</selfCollide>
 		</gazebo>
 		<gazebo reference="${name}_4_link">
-			<material value="Schunk/LightGrey" />
+			<material>Schunk/LightGrey</material>
 			<turnGravityOff>false</turnGravityOff>
             <selfCollide>true</selfCollide>
 		</gazebo>
 		<gazebo reference="${name}_5_link">
-			<material value="Schunk/Blue" />
+			<material>Schunk/Blue</material>
 			<turnGravityOff>false</turnGravityOff>
             <selfCollide>true</selfCollide>
 		</gazebo>
 		<gazebo reference="${name}_6_link">
-			<material value="Schunk/LightGrey" />
+			<material>Schunk/LightGrey</material>
 			<turnGravityOff>false</turnGravityOff>
             <selfCollide>true</selfCollide>

File: crom_description/urdf/arms/lwa4p/lwa4p.urdf.xacro (robot description, xacro)
@@ -3,4 +3,6 @@
 	<xacro:include filename="$(find crom_description)/urdf/arms/lwa4p/lwa4p.gazebo.xacro" />
 	<xacro:include filename="$(find crom_description)/urdf/arms/lwa4p/lwa4p.transmission.xacro" />
+	 <!-- calibration -->
+    <xacro:include filename="$(find crom_description)/urdf/arms/lwa4p/calibration.urdf.xacro" />
 	<xacro:property name="joint_1_upper_limit" value="2.967059678" /> <!-- 170º -->
 	<xacro:property name="joint_1_lower_limit" value="-2.967059678" /> <!-- -170º -->
@@ -39,5 +41,5 @@
 					<mesh filename="package://crom_description/meshes/arms/lwa4p/stl/arm_base.stl" />
 				</geometry>
-				<material name="Schunk/LightGrey" />
+				<material name="schunk_light_grey" />
 			</visual>
 			<collision>
@@ -70,5 +72,5 @@
 					<mesh filename="package://crom_description/meshes/arms/lwa4p/stl/arm_1_link.stl" />
 				</geometry>
-				<material name="Schunk/Blue" />
+				<material name="schunk_light_grey" />
 			</visual>
 			<collision>
@@ -101,5 +103,5 @@
 					<mesh filename="package://crom_description/meshes/arms/lwa4p/stl/arm_2_link.stl" />
 				</geometry>
-				<material name="Schunk/LightGrey" />
+				<material name="schunk_blue" />
 			</visual>
 			<collision>
@@ -132,5 +134,5 @@
 					<mesh filename="package://crom_description/meshes/arms/lwa4p/stl/arm_3_link.stl" />
 				</geometry>
-				<material name="Schunk/Blue" />
+				<material name="schunk_light_grey" />
 			</visual>
 			<collision>
@@ -163,5 +165,5 @@
 					<mesh filename="package://crom_description/meshes/arms/lwa4p/stl/arm_4_link.stl" />
 				</geometry>
-				<material name="Schunk/LightGrey" />
+				<material name="schunk_blue" />
 			</visual>
 			<collision>
@@ -194,5 +196,5 @@
 					<mesh filename="package://crom_description/meshes/arms/lwa4p/stl/arm_5_link.stl" />
 				</geometry>
-				<material name="Schunk/Blue" />
+				<material name="schunk_light_grey" />
 			</visual>
 			<collision>
@@ -225,5 +227,5 @@
 					<mesh filename="package://crom_description/meshes/arms/lwa4p/stl/arm_6_link.stl" />
 				</geometry>
-				<material name="Schunk/LightGrey" />
+				<material name="schunk_light_grey" />
 			</visual>
 			<collision>

File: crom_description/urdf/arms/lwa4p/materials.urdf.xacro (robot description, xacro)
@@ -1,17 +1,17 @@
 <?xml version="1.0"?>
 <robot>
-	<material name="Schunk/LightGrey">
+	<material name="schunk_light_grey">
 		<color rgba="0.7 0.7 0.7 1.0"/>
 	</material>
-	<material name="Schunk/DarkGrey">
+	<material name="schunk_dark_grey">
 		<color rgba="0.4 0.4 0.4 1.0"/>
 	</material>
-	<material name="Schunk/Black">
+	<material name="schunk_black">
 		<color rgba="0.0 0.0 0.0 1.0"/>
 	</material>
-	<material name="Schunk/DarkGolden">
+	<material name="schunk_dark_golden">
 		<color rgba="0.4 0.4 0.3 1.0"/>
 	</material>
-	<material name="Schunk/Blue">
+	<material name="schunk_blue">
 		<color rgba="0.0 0.0 0.8 1.0"/>
 	</material>

File: crom_description/urdf/robot/crom.urdf.xacro (robot description, xacro)
@@ -4,6 +4,4 @@
   <xacro:include filename="$(find crom_description)/urdf/robot/crom.gazebo" />
   <xacro:include filename="$(find crom_description)/urdf/arms/lwa4p/materials.urdf.xacro" />
-  <!-- calibration -->
-  <xacro:include filename="$(find crom_description)/urdf/arms/lwa4p/calibration.urdf.xacro" />
   <!-- schunk powerball -->
   <xacro:include filename="$(find crom_description)/urdf/arms/lwa4p/lwa4p.urdf.xacro" />
@@ -87,14 +85,12 @@
 		   <origin xyz="0 0 0" rpy="0 0 0" />
 		   <geometry>
-			 <mesh filename="package://crom_description/meshes/torso/torso_body.dae"/>
-		   </geometry>
-		<material name="Red">
-			<color rgba="0.3 0.3 0.3 1"/>
-			</material>
-		</visual>
-		<collision>
-		   <origin xyz="0 0 0" rpy="0 0 0" />
-		   <geometry>
-			 <mesh filename="package://crom_description/meshes/torso/torso_body.dae"/>
+			 <mesh filename="package://crom_description/meshes/torso/torso_body.stl"/>
+		   </geometry>
+		   <material name="schunk_blue"/>
+		</visual>
+		<collision>
+		   <origin xyz="0 0 0" rpy="0 0 0" />
+		   <geometry>
+			 <mesh filename="package://crom_description/meshes/torso/torso_body.stl"/>
 		   </geometry>
 		</collision>
