Commit message: crom_description:lwa4p.urdf.xacro: replacing .stl by .dae in collision tag

File: crom_description/urdf/arms/lwa4p/lwa4p.urdf.xacro (robot description, xacro)
@@ -46,5 +46,5 @@
 				<origin xyz="0 0 0" rpy="0 0 0" />
 				<geometry>
-					<mesh filename="package://crom_description/meshes/arms/lwa4p/stl/arm_base.stl" />
+					<mesh filename="package://crom_description/meshes/arms/lwa4p/dae/arm_base.dae" />
 				</geometry>
 			</collision>
@@ -77,5 +77,5 @@
 				<origin xyz="0 0 0" rpy="0 0 0" />
 				<geometry>
-					<mesh filename="package://crom_description/meshes/arms/lwa4p/stl/arm_1_link.stl" />
+					<mesh filename="package://crom_description/meshes/arms/lwa4p/dae/arm_1_link.dae" />
 				</geometry>
 			</collision>
@@ -108,5 +108,5 @@
 				<origin xyz="0 0 0" rpy="0 0 0" />
 				<geometry>
-					<mesh filename="package://crom_description/meshes/arms/lwa4p/stl/arm_2_link.stl" />
+					<mesh filename="package://crom_description/meshes/arms/lwa4p/dae/arm_2_link.dae" />
 				</geometry>
 			</collision>
@@ -139,5 +139,5 @@
 				<origin xyz="0 0 0" rpy="0 0 0" />
 				<geometry>
-					<mesh filename="package://crom_description/meshes/arms/lwa4p/stl/arm_3_link.stl" />
+					<mesh filename="package://crom_description/meshes/arms/lwa4p/dae/arm_3_link.dae" />
 				</geometry>
 			</collision>
@@ -170,5 +170,5 @@
 				<origin xyz="0 0 0" rpy="0 0 0" />
 				<geometry>
-					<mesh filename="package://crom_description/meshes/arms/lwa4p/stl/arm_4_link.stl" />
+					<mesh filename="package://crom_description/meshes/arms/lwa4p/dae/arm_4_link.dae" />
 				</geometry>
 			</collision>
@@ -201,5 +201,5 @@
 				<origin xyz="0 0 0" rpy="0 0 0" />
 				<geometry>
-					<mesh filename="package://crom_description/meshes/arms/lwa4p/stl/arm_5_link.stl" />
+					<mesh filename="package://crom_description/meshes/arms/lwa4p/dae/arm_5_link.dae" />
 				</geometry>
 			</collision>
@@ -232,5 +232,5 @@
 				<origin xyz="0 0 0" rpy="0 0 0" />
 				<geometry>
-					<mesh filename="package://crom_description/meshes/arms/lwa4p/stl/arm_6_link.stl" />
+					<mesh filename="package://crom_description/meshes/arms/lwa4p/dae/arm_6_link.dae" />
 				</geometry>
 			</collision>
