Commit message: crom_description: setting colors for RVIZ and Gazebo

File: crom_description/robots/crom.urdf.xacro (robot description, xacro)
@@ -2,5 +2,5 @@
 <robot name="crom" xmlns:xacro="http://www.ros.org/wiki/xacro">
   <!-- Import all Gazebo-customization elements, including Gazebo colors -->
-  <xacro:include filename="$(find crom_description)/urdf/robot/crom.gazebo" />
+  <xacro:include filename="$(find crom_description)/robots/crom.gazebo" />
   <xacro:include filename="$(find crom_description)/urdf/arms/lwa4p/materials.urdf.xacro" />
   <!-- schunk powerball -->
@@ -65,11 +65,12 @@
 		   <origin xyz="0 0 0" rpy="0 0 0" />
 		   <geometry>
-		 <mesh filename="package://crom_description/meshes/torso/torso_base.dae"/>
-		   </geometry>
-		</visual>
-		<collision>
-		   <origin xyz="0 0 0" rpy="0 0 0 " />
-		   <geometry>
-			 <mesh filename="package://crom_description/meshes/torso/torso_base.dae"/>
+		     <mesh filename="package://crom_description/meshes/torso/torso_base.stl"/>
+		   </geometry>
+		   <material name="schunk_black"/>
+		</visual>
+		<collision>
+		   <origin xyz="0 0 0" rpy="0 0 0 " />
+		   <geometry>
+			 <mesh filename="package://crom_description/meshes/torso/torso_base.stl"/>
 		   </geometry>
 		</collision>

File: crom_description/urdf/arms/lwa4p/lwa4p.gazebo.xacro (robot description, xacro)
@@ -3,35 +3,35 @@
 	<xacro:macro name="schunk_lwa4p_gazebo" params="name">
 		<gazebo reference="${name}_0_link">
-			<material>Schunk/LightGrey</material>
+			<material>Gazebo/Grey</material>
 			<turnGravityOff>false</turnGravityOff>
             <selfCollide>true</selfCollide>
 		</gazebo>
 		<gazebo reference="${name}_1_link">
-			<material>Schunk/Blue</material>
+			<material>Gazebo/Grey</material>
 			<turnGravityOff>false</turnGravityOff>
             <selfCollide>true</selfCollide>
 		</gazebo>
 		<gazebo reference="${name}_2_link">
-			<material>Schunk/LightGrey</material>
+			<material>Gazebo/Blue</material>
 			<turnGravityOff>false</turnGravityOff>
             <selfCollide>true</selfCollide>
 		</gazebo>
 		<gazebo reference="${name}_3_link">
-			<material>Schunk/Blue</material>
+			<material>Gazebo/Grey</material>
 			<turnGravityOff>false</turnGravityOff>
              <selfCollide>true</selfCollide>
 		</gazebo>
 		<gazebo reference="${name}_4_link">
-			<material>Schunk/LightGrey</material>
+			<material>Gazebo/Blue</material>
 			<turnGravityOff>false</turnGravityOff>
             <selfCollide>true</selfCollide>
 		</gazebo>
 		<gazebo reference="${name}_5_link">
-			<material>Schunk/Blue</material>
+			<material>Gazebo/Grey</material>
 			<turnGravityOff>false</turnGravityOff>
             <selfCollide>true</selfCollide>
 		</gazebo>
 		<gazebo reference="${name}_6_link">
-			<material>Schunk/LightGrey</material>
+			<material>Gazebo/Grey</material>
 			<turnGravityOff>false</turnGravityOff>
             <selfCollide>true</selfCollide>

Commit message: crom_description: moving kinect and head cameras to head urdf/gazebo description

File: crom_description/robots/crom.urdf.xacro (robot description, xacro)
@@ -10,5 +10,4 @@
   <!-- Head -->
   <xacro:include filename="$(find crom_description)/urdf/head/head.urdf.xacro"/>
-  <xacro:include filename="$(find crom_description)/urdf/head/head.gazebo" />
   <!-- WSG50 GRIPPER -->
   <xacro:include filename="$(find crom_description)/urdf/grippers/wsg50/wsg50.urdf.xacro" />
@@ -221,5 +220,4 @@
 	</link>
 	<joint name="camera_2_hand_left_joint" type="fixed">
-		<!--origin xyz="0 0 0" rpy="0 0.26 ${PI}" /-->
 		<origin xyz="0 0 0" rpy="0 -${PI_2} 0" />
 		<parent link="camera_1_hand_left_link"/>
@@ -230,5 +228,4 @@
 	</link>
 	<joint name="hand_right_base_joint" type="fixed">
-		<!--origin xyz="0 0 0.085" rpy="0 0 1.5708" /-->
 		<origin xyz="0 0 0.085" rpy="1.5708 -1.5708 0.0" />
 		<parent link="right_arm_6_link"/>
@@ -243,5 +240,4 @@
 	</link>
 	<joint name="hand_right_grasp_joint" type="fixed">
-		<!--origin xyz="0 0 0.085" rpy="0 0 1.5708" /-->
 		<origin xyz="0.14 0 0" rpy="0.0 0.0 0.0" />
 		<parent link="hand_right_base_link"/>
@@ -251,5 +247,4 @@
 	<link name="camera_1_hand_right_link"/>
 	<joint name="camera_1_hand_right_joint" type="fixed">
-		<!--origin xyz="0 0.055 0.045" rpy="-1.5708 -1.5708 0.0" /-->
 		<origin xyz="0.045 0.055 0.0" rpy="-1.5708 0.0 0.0" />
 		<parent link="hand_right_base_link"/>

File: crom_description/urdf/head/head.urdf.xacro (robot description, xacro)
@@ -1,4 +1,6 @@
 <?xml version="1.0"?>
 <robot xmlns:xacro="http://www.ros.org/wiki/xacro">
+	<xacro:include filename="$(find crom_description)/urdf/head/head.gazebo" />
+	<xacro:include filename="$(find crom_description)/urdf/head/kinect.urdf.xacro" />
 	<!-- Robot mechanical and motor parameters -->
 	<xacro:property name="PI" value="3.1415926535897931"/>
@@ -193,20 +195,9 @@
 			<axis xyz="0 0 1" rpy="0 0 0" />
 		</joint>
-		<!--link name="${name}_kinect_frame_link">
-			<inertial>
-				<mass value="0.01" />
-				<origin xyz="0 0 0" />
-			<inertia  ixx="0.059" ixy="0.0"  ixz="0.0"  iyy="0.055"  iyz="0.0"  izz="0.059" />
-		</inertial>
-		</link>
-		<joint name="${name}_kinect_frame_joint" type="fixed">
-			<parent link="${name}_kinect_link"/>
-			<child link="${name}_kinect_frame_link"/>
-			<origin xyz="0.5 0 0" rpy="0 1.57 1.57" />
-			<axis xyz="0 0 1" rpy="0 0 0" />
-		</joint-->
 		<!-- Import all Gazebo-customization elements, including Gazebo colors -->
-		<!--include filename="$(find robotnik_torso_description)/urdf/head.gazebo" /-->
 		<xacro:head_gazebo name="${name}" />
+		<xacro:sensor_kinect name="kinect" parent="${name}_kinect_link">
+			<origin xyz="0.0 0 0.0365" rpy="0 0 0"/>
+		</xacro:sensor_kinect>
 	</xacro:macro>
 </robot>

Commit message: crom_description: adding urdf model and launch file for the arm and gripper

File: crom_description/robots/crom.urdf.xacro (robot description, xacro)
@@ -24,9 +24,9 @@
   <xacro:property name="waist_mechanical_reduction" value="1.0" />
   <!-- Used for fixing robot to Gazebo 'base_link' -->
-  <link name="world"/>
+  <!--link name="world"/>
   <joint name="fixed" type="fixed">
 	<parent link="world"/>
 	<child link="base_footprint"/>
-  </joint>
+  </joint-->
   <!-- BASE FOOTPRINT -->
   <!-- base_footprint is a fictitious link(frame) that is on the ground right below base_link origin,
@@ -57,5 +57,5 @@
 	<link name="base_link">
 		<inertial>
-		  <mass value="50.0" />
+		  <mass value="400.0" />
 		  <origin xyz="0 0 0" />
 		  <inertia  ixx="3.737" ixy="0.008"  ixz="-0.144"  iyy="8.311"  iyz="-0.004"  izz="8.893" />
@@ -233,6 +233,6 @@
 	</joint>
 	<!-- WSG50 GRIPPER -->
-	<xacro:wsg50 name="wsg50" parent="hand_right_base_link">
-		<origin xyz="0 0 0" rpy="0 1.5708 0" />
+	<xacro:wsg50 name="wsg50" parent="right_arm_6_link">
+		<origin xyz="0 0 0.085" rpy="0 0 1.5708" />
 	</xacro:wsg50>
 	<!-- Grasp link GRIPPER on right arm -->

Commit message: crom_description:crom.urdf: replacing .stl by .dae in collision tag

File: crom_description/robots/crom.urdf.xacro (robot description, xacro)
@@ -57,5 +57,5 @@
 	<link name="base_link">
 		<inertial>
-		  <mass value="400.0" />
+		  <mass value="800.0" />
 		  <origin xyz="0 0 0" />
 		  <inertia  ixx="3.737" ixy="0.008"  ixz="-0.144"  iyy="8.311"  iyz="-0.004"  izz="8.893" />
@@ -71,5 +71,5 @@
 		   <origin xyz="0 0 0" rpy="0 0 0 " />
 		   <geometry>
-			 <mesh filename="package://crom_description/meshes/torso/torso_base.stl"/>
+			 <mesh filename="package://crom_description/meshes/torso/torso_base.dae"/>
 		   </geometry>
 		</collision>
@@ -92,5 +92,5 @@
 		   <origin xyz="0 0 0" rpy="0 0 0" />
 		   <geometry>
-			 <mesh filename="package://crom_description/meshes/torso/torso_body.stl"/>
+			 <mesh filename="package://crom_description/meshes/torso/torso_body.dae"/>
 		   </geometry>
 		</collision>
@@ -193,6 +193,6 @@
 	<joint name="hand_left_grasp_joint" type="fixed">
 		<!--origin xyz="0 0 0.085" rpy="0 0 1.5708" /-->
-		<origin xyz="0 0 0.10" rpy="0.0 0.0 0.0" />
-		<parent link="hand_left_base_link"/>
+		<origin xyz="0 0 0.212" rpy="0.0 0.0 0.0" />
+		<parent link="left_arm_6_link"/>
 		<child link="hand_left_grasp_link"/>
 	</joint>

Commit message: crom_description: Adding Robotnik's logo to the robot

File: crom_description/robots/crom.urdf.xacro (robot description, xacro)
@@ -116,4 +116,21 @@
 		</actuator>
 	</transmission>
+   <!-- LOGO -->
+   <link name="logo_link">
+		<visual>
+		   <origin xyz="0.0 0 0.0" rpy="0 0 0" />
+		   <geometry>
+			 <mesh filename="package://crom_description/meshes/torso/torso_logo.dae"/>
+		   </geometry>
+		   <material name="red">
+			 <color rgba="0.8 0.1 0.1 1"/>
+		   </material>
+		</visual>
+	</link>
+	<joint name="logo_joint" type="fixed">
+		<parent link="waist_link"/>
+		<child link="logo_link"/>
+		<origin xyz="0.002 0 0" rpy="0 0 0" />
+	</joint>
   	<!-- LEFT ARM -->
   	<link name="powerball_left_base_link">
